Commit message: update urdf description

File: rangerboxcr10lidar_description/urdf/RangerCR10LiDAR.urdf (robot description, URDF)
Before this commit: robot RangerCR10LiDAR, 52 links, 51 joints
Links:
- link base_link: geometry collision mesh filename=package://rangerboxcr10lidar_description/meshes/ranger_mesh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; visual mesh filename=package://rangerboxcr10lidar_description/meshes/ranger_mesh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
- link box_link: geometry collision mesh filename=package://rangerboxcr10lidar_description/meshes/box_link.STL; visual mesh filename=package://rangerboxcr10lidar_description/meshes/box_link.STL
- link cr10_Link1: geometry collision mesh filename=package://rangerboxcr10lidar_description/meshes/cr10_meshes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; visual mesh filename=package://rangerboxcr10lidar_description/meshes/cr10_meshes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
- link cr10_Link2: geometry collision mesh filename=package://rangerboxcr10lidar_description/meshes/cr10_meshes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; visual mesh filename=package://rangerboxcr10lidar_description/meshes/cr10_meshes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
- link cr10_Link3: geometry collision mesh filename=package://rangerboxcr10lidar_description/meshes/cr10_meshes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; visual mesh filename=package://rangerboxcr10lidar_description/meshes/cr10_meshes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
- link cr10_Link4: geometry collision mesh filename=package://rangerboxcr10lidar_description/meshes/cr10_meshes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; visual mesh filename=package://rangerboxcr10lidar_description/meshes/cr10_meshes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
- link cr10_Link5: geometry collision mesh filename=package://rangerboxcr10lidar_description/meshes/cr10_meshes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; visual mesh filename=package://rangerboxcr10lidar_description/meshes/cr10_meshes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
- link cr10_Link6: geometry collision mesh filename=package://rangerboxcr10lidar_description/meshes/cr10_meshes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; visual mesh filename=package://rangerboxcr10lidar_description/meshes/cr10_meshes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
- link cr10_base_link: geometry collision mesh filename=package://rangerboxcr10lidar_description/meshes/cr10_meshes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; visual mesh filename=package://rangerboxcr10lidar_description/meshes/cr10_meshes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
- link d435_link: geometry collision box size=0.02505 0.090 0.025; visual mesh filename=package://rangerboxcr10lidar_description/meshes/realsense_m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 scale=1 1 1
- link d455_link: geometry collision box size=0.026 0.124 0.029; visual mesh filename=package://rangerboxcr10lidar_description/meshes/realsense_m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 scale=0.001 0.001 0.001
- link fl_steering_wheel_link: geometry collision mesh filename=package://rangerboxcr10lidar_description/meshes/ranger_mesh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; visual mesh filename=package://rangerboxcr10lidar_description/meshes/ranger_mesh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
- link fl_wheel_link: geometry collision mesh filename=package://rangerboxcr10lidar_description/meshes/ranger_mesh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; visual mesh filename=package://rangerboxcr10lidar_description/meshes/ranger_mesh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
- link fr_steering_link: geometry collision mesh filename=package://rangerboxcr10lidar_description/meshes/ranger_mesh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; visual mesh filename=package://rangerboxcr10lidar_description/meshes/ranger_mesh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
- link fr_wheel_link: geometry collision mesh filename=package://rangerboxcr10lidar_description/meshes/ranger_mesh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; visual mesh filename=package://rangerboxcr10lidar_description/meshes/ranger_mesh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
- link gripper_base_link: geometry collision mesh filename=package://rangerboxcr10lidar_description/meshes/ag95_meshes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 scale=0.001 0.001 0.001; visual mesh filename=package://rangerboxcr10lidar_description/meshes/ag95_meshes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 scale=0.001 0.001 0.001
- link gripper_finger1_finger_link: geometry collision mesh filename=package://rangerboxcr10lidar_description/meshes/ag95_meshes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 scale=0.001 0.001 0.001; visual mesh filename=package://rangerboxcr10lidar_description/meshes/ag95_meshes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 scale=0.001 0.001 0.001
- link gripper_finger1_finger_tip_link: geometry collision mesh filename=package://rangerboxcr10lidar_description/meshes/ag95_meshes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 scale=0.001 0.001 0.001; visual mesh filename=package://rangerboxcr10lidar_description/meshes/ag95_meshes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 scale=0.001 0.001 0.001
- link gripper_finger1_inner_knuckle_link: geometry collision mesh filename=package://rangerboxcr10lidar_description/meshes/ag95_meshes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 scale=0.001 0.001 0.001; visual mesh filename=package://rangerboxcr10lidar_description/meshes/ag95_meshes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 scale=0.001 0.001 0.001
- link gripper_finger1_knuckle_link: geometry collision mesh filename=package://rangerboxcr10lidar_description/meshes/ag95_meshes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 scale=0.001 0.001 0.001; visual mesh filename=package://rangerboxcr10lidar_description/meshes/ag95_meshes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 scale=0.001 0.001 0.001
- link gripper_finger2_finger_link: geometry collision mesh filename=package://rangerboxcr10lidar_description/meshes/ag95_meshes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 scale=0.001 0.001 0.001; visual mesh filename=package://rangerboxcr10lidar_description/meshes/ag95_meshes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 scale=0.001 0.001 0.001
- link gripper_finger2_finger_tip_link: geometry collision mesh filename=package://rangerboxcr10lidar_description/meshes/ag95_meshes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 scale=0.001 0.001 0.001; visual mesh filename=package://rangerboxcr10lidar_description/meshes/ag95_meshes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 scale=0.001 0.001 0.001
- link gripper_finger2_inner_knuckle_link: geometry collision mesh filename=package://rangerboxcr10lidar_description/meshes/ag95_meshes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 scale=0.001 0.001 0.001; visual mesh filename=package://rangerboxcr10lidar_description/meshes/ag95_meshes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 scale=0.001 0.001 0.001
- link gripper_finger2_knuckle_link: geometry collision mesh filename=package://rangerboxcr10lidar_description/meshes/ag95_meshes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 scale=0.001 0.001 0.001; visual mesh filename=package://rangerboxcr10lidar_description/meshes/ag95_meshes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 scale=0.001 0.001 0.001
- link lidar_link0: geometry collision mesh filename=package://rangerboxcr10lidar_description/meshes/lidar_link0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; visual mesh filename=package://rangerboxcr10lidar_description/meshes/lidar_link0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
- link rl_steering_wheel_link: geometry collision mesh filename=package://rangerboxcr10lidar_description/meshes/ranger_mesh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; visual mesh filename=package://rangerboxcr10lidar_description/meshes/ranger_mesh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
- link rl_wheel_link: geometry collision mesh filename=package://rangerboxcr10lidar_description/meshes/ranger_mesh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; visual mesh filename=package://rangerboxcr10lidar_description/meshes/ranger_mesh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
- link rr_steering_wheel_link: geometry collision mesh filename=package://rangerboxcr10lidar_description/meshes/ranger_mesh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; visual mesh filename=package://rangerboxcr10lidar_description/meshes/ranger_mesh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
- link rr_wheel_link: geometry collision mesh filename=package://rangerboxcr10lidar_description/meshes/ranger_mesh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; visual mesh filename=package://rangerboxcr10lidar_description/meshes/ranger_mesh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
