Commit message: Update package metadata, refine URDF structure, and add RViz configuration
- Updated author and maintainer information in package.xml.
- Refined the URDF structure by removing unnecessary comments and ensuring consistent formatting.
- Adjusted joint limits and parameters for gripper joints in the URDF.
- Added a new RViz configuration file for visualizing the robot model.

File: rangerboxcr10lidar_description/urdf/rangercr10lidar.urdf (robot description, URDF)
Before this commit: robot rangercr10lidar, 52 links, 51 joints
Joints:
- joint gripper_finger1_finger_tip_joint: origin xyz=0.0394969463769 0.0 0.0382752038125  rpy=0.0 0.0 0.0 -> xyz=0.0394969463769 0.0 0.0382752038125 rpy=0.0 0.0 0.0
- joint gripper_finger2_finger_tip_joint: origin xyz=0.0394969463769  0.0 0.0382752038125   rpy=0.0 0.0 0.0 -> xyz=0.0394969463769 0.0 0.0382752038125 rpy=0.0 0.0 0.0
- joint gripper_finger2_joint: limit lower=-3.14 upper=3.14 effort=1000 velocity=100.0 -> lower=0.0 upper=0.6524 effort=1000 velocity=2.0; mimic joint=gripper_finger1_joint -> joint=gripper_finger1_joint multiplier=1.0 offset=0; origin xyz=0.016  0 0.10586  rpy=0.0 0.0 0.0 -> xyz=0.016 0 0.10586 rpy=0.0 0.0 0.0
